File: kicad/RDS-2P Плата питания/RDS-2P Плата питания.kicad_pcb (KiCad board)
At the start: 2 copper layers, 100 x 100 mm, 13 parts, among them J1 XT30U, J2 XT30U2, J3 ЗАР, J4 ВЫКЛ, J5 8.4V, J6 8.4V, J7 5V, J8 ИНД, U1 Converter_Mini560, U2 BMS_2S_20A

Commit message: Update RDS-2P Плата питания.kicad_pcb
Добавил отверстия под винты для присоединения платы к RDS-2P
Parts:
- added Hole_gge19008: Hole_gge19008, Плата питания для RDS-2P:Hole_gge19008, F.Cu at (150.0, 110.0)
- added Hole_gge19023: Hole_gge19023, Плата питания для RDS-2P:Hole_gge19023, F.Cu at (102.0, 110.0)
- added Pad_gge17218: Pad_gge17218, Плата питания для RDS-2P:Pad_gge17218, F.Cu at (102.0, 110.0)
- added Pad_gge17221: Pad_gge17221, Плата питания для RDS-2P:Pad_gge17221, F.Cu at (150.0, 110.0)

Commit message: Fix Отверстий RDS-2P Плата питания.kicad_pcb
Убрал ошибки компилятора по поводу отверстий
Parts:
- removed Hole_gge19008: Hole_gge19008, Плата питания для RDS-2P:Hole_gge19008
- removed Hole_gge19023: Hole_gge19023, Плата питания для RDS-2P:Hole_gge19023
Changed lines of the file:
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@@
 			)
 		)
-		(pad "4" thru_hole oval
+		(pad "" np_thru_hole oval
 			(at 0 0)
 			(size 1.524 1.524)
 			(drill 3)
 			(layers "*.Cu" "*.Mask")
-			(remove_unused_layers no)
 			(solder_mask_margin 0.0508)
 			(solder_paste_margin 0)
@@
 			)
 		)
-		(pad "3" thru_hole oval
+		(pad "" np_thru_hole oval
 			(at 0 0)
 			(size 1.524 1.524)
 			(drill 3)
 			(layers "*.Cu" "*.Mask")
-			(remove_unused_layers no)
 			(solder_mask_margin 0.0508)
 			(solder_paste_margin 0)
 			(thermal_bridge_angle 0)
-		)
-		(embedded_fonts no)
-	)
-	(footprint "Плата питания для RDS-2P:Hole_gge19023"
-		(layer "F.Cu")
-		(at 102 110)
-		(property "Reference" "Hole_gge19023"
-			(at 0 0 0)
-			(layer "F.SilkS")
-			(hide yes)
-			(effects
-				(font
-					(size 0.5 0.5)
-					(thickness 0.15)
-				)
-			)
-		)
-		(property "Value" "Hole_gge19023"
-			(at 0 0 0)
-			(layer "F.Fab")
-			(hide yes)
-			(effects
-				(font
-					(size 0.5 0.5)
-					(thickness 0.15)
-				)
-			)
-		)
-		(property "Datasheet" ""
-			(at 0 0 0)
-			(layer "F.Fab")
-			(hide yes)
-			(effects
-				(font
-					(size 1.27 1.27)
-					(thickness 0.15)
-				)
-			)
-		)
-		(property "Description" ""
-			(at 0 0 0)
-			(layer "F.Fab")
-			(hide yes)
-			(effects
-				(font
-					(size 1.27 1.27)
-					(thickness 0.15)
-				)
-			)
-		)
-		(pad "" np_thru_hole circle
-			(at 0 0)
-			(size 3 3)
-			(drill 3)
-			(layers "*.Cu" "*.Mask")
 		)
 		(embedded_fonts no)
@@
 		)
 	)
-	(footprint "Плата питания для RDS-2P:Hole_gge19008"
-		(layer "F.Cu")
-		(at 149.9605 109.9606)
-		(property "Reference" "Hole_gge19008"
-			(at 0 0 0)
-			(layer "F.SilkS")
-			(hide yes)
-			(effects
-				(font
-					(size 0.5 0.5)
-					(thickness 0.15)
-				)
-			)
-		)
-		(property "Value" "Hole_gge19008"
-			(at 0 0 0)
-			(layer "F.Fab")
-			(hide yes)
-			(effects
-				(font
-					(size 0.5 0.5)
-					(thickness 0.15)
-				)
-			)
-		)
-		(property "Datasheet" ""
-			(at 0 0 0)
-			(layer "F.Fab")
-			(hide yes)
-			(effects
-				(font
-					(size 1.27 1.27)
-					(thickness 0.15)
-				)
-			)
-		)
-		(property "Description" ""
-			(at 0 0 0)
-			(layer "F.Fab")
-			(hide yes)
-			(effects
-				(font
-					(size 1.27 1.27)
-					(thickness 0.15)
-				)
-			)
-		)
-		(pad "" np_thru_hole circle
-			(at 0 0)
-			(size 3 3)
-			(drill 3)
-			(layers "*.Cu" "*.Mask")
-		)
-		(embedded_fonts no)
-	)
 	(footprint "Connector_AMASS:AMASS_XT30U-power_1x02_P5.0mm_Vertical"
