File: kicad/RDS-2P Плата коммутации двигателей/RDS-2P Плата коммутации двигателей.kicad_sch (KiCad schematic)
At the start: 10 parts, among them J1 XT30U, J2 XT30U, J3 5264-3AW, J4 5264-3AW, J5 5264-3AW, J6 5264-3AW, J7 Conn_01x01_Pin, J8 Conn_01x01_Pin, J9 Conn_01x01_Pin, U1 Converter_Mini560

Commit message: Fix: pinout Mini560
Исправил распиновку Mini560 на платах
Connections:
- net +8.4V: no longer U1.5 (EN)
- new net 0 1: U1.5 (EN)
Changed lines of the file:
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@@
 		(color 255 0 13 1)
 	)
-	(junction
-		(at 114.3 71.12)
-		(diameter 0)
-		(color 0 0 0 0)
-	)
 	(wire
 		(pts
@@
 	(wire
 		(pts
-			(xy 114.3 71.12) (xy 118.11 71.12)
-		)
-		(stroke
-			(width 0)
-			(type default)
-			(color 255 0 13 1)
-		)
-	)
-	(wire
-		(pts
 			(xy 121.92 88.9) (xy 127 88.9)
 		)
@@
 	(wire
 		(pts
-			(xy 114.3 93.98) (xy 114.3 71.12)
+			(xy 114.3 66.04) (xy 114.3 93.98)
 		)
 		(stroke
@@
 	(wire
 		(pts
-			(xy 114.3 71.12) (xy 114.3 66.04)
-		)
-		(stroke
-			(width 0)
-			(type default)
-			(color 255 0 13 1)
-		)
-	)
-	(wire
-		(pts
 			(xy 116.84 96.52) (xy 116.84 102.87)
 		)
@@
 	(wire
 		(pts
+			(xy 106.68 71.12) (xy 118.11 71.12)
+		)
+		(stroke
+			(width 0)
+			(type default)
+		)
+	)
+	(wire
+		(pts
 			(xy 106.68 93.98) (xy 113.03 93.98)
 		)
@@
 		)
 	)
+	(symbol
+		(lib_id "Simulation_SPICE:0")
+		(at 106.68 71.12 270)
+		(unit 1)
+		(exclude_from_sim no)
+		(in_bom yes)
+		(on_board yes)
+		(dnp no)
+		(fields_autoplaced yes)
+		(property "Reference" "#GND02"
+			(at 101.6 71.12 0)
+			(effects
+				(font
+					(size 1.27 1.27)
+				)
+				(hide yes)
+			)
+		)
+		(property "Value" "0 1"
+			(at 107.95 71.1199 90)
+			(effects
+				(font
+					(size 1.27 1.27)
+				)
+				(justify left)
+			)
+		)
+		(property "Footprint" ""
+			(at 106.68 71.12 0)
+			(effects
+				(font
+					(size 1.27 1.27)
+				)
+				(hide yes)
+			)
+		)
+		(property "Datasheet" "https://ngspice.sourceforge.io/docs/ngspice-html-manual/manual.xhtml#subsec_Circuit_elements__device"
+			(at 96.52 71.12 0)
+			(effects
+				(font
+					(size 1.27 1.27)
+				)
+				(hide yes)
+			)
+		)
+		(property "Description" "0V reference potential for simulation"
+			(at 99.06 71.12 0)
+			(effects
+				(font
+					(size 1.27 1.27)
+				)
+				(hide yes)
+			)
+		)
+		(pin "1"
+		)
+		(instances
+			(project ""
+				(path "/f73a4416-8a7c-4278-9d1a-922baee4e7ea"
+					(reference "#GND02")
+					(unit 1)
+				)
+			)
+		)
+	)
